File: fpga-mgt.kicad_sch (KiCad schematic)
At the start: 11 parts, among them U4 XC7K160T-FFG676

Commit message: Removing PCIe from sch and PCB
Parts:
- removed C222, C223, C226, C227, C228, C229, C230, C231, C232, C233: C_100n_0402, antmicro-footprints:C_0402_1005Metric, symbol antmicroCapacitors0402:C_100n_0402
- removed U4: XC7K160T-FFG676, antmicro-footprints:BGA-676_27x27mm_Layout26x26_P1x1mm_FFG676, symbol antmicroFPGAChips:XC7K160T-FFG676
Connections:
- no-connect marks 22 -> 0
Other:
- note removed: "BANK 115"
- note removed: "BANK 116"
- note removed: "MGT Interface"
- note removed: "Place capacitors close to connector"
