File: hdmi-sd-card.kicad_sch (KiCad schematic)
At the start: 33 parts, among them J4 HDMI-A_WE_685119134923, J5 MicroSD_693071020811, U10 TPD4E05U06QDQARQ1, U11 TPD4E05U06QDQARQ1, U12 TPD4E05U06QDQARQ1, U14 TPD4E05U06QDQARQ1

Commit message: Removing HDMI from sch and PCB
Parts:
- removed C126: C_10u_6.3V_0402, antmicro-footprints:C_0402_1005Metric, symbol antmicroCapacitors0402:C_10u_6.3V_0402
- removed C132: C_100n_0402, antmicro-footprints:C_0402_1005Metric, symbol antmicroCapacitors0402:C_100n_0402
- removed D14: BAT54-02V-G3-08, antmicro-footprints:SOD-523, symbol antmicroDiodesRectifiersSingle:BAT54-02V-G3-08
- removed FB3: FB_120Z_2A_Murata-BLM18PG_0603, antmicro-footprints:FB_0603_1608Metric, symbol antmicroFerriteBeadsandChips:FB_120Z_2A_Murata-BLM18PG_0603
- removed J4: HDMI-A_WE_685119134923, antmicro-footprints:HDMI-A_Receptacle_WE_685119134923, symbol antmicroVideoConnectors:HDMI-A_WE_685119134923
- removed R70, R71, R72, R73, R74, R75, R76, R77: R_0R_0402, antmicro-footprints:R_0402_1005Metric, symbol antmicroResistors0402:R_0R_0402
- removed R89: R_330R_0402, antmicro-footprints:R_0402_1005Metric, symbol antmicroResistors0402:R_330R_0402
- removed TP2, TP3, TP4, TP5, TP6: TP_1mm_SMD, antmicro-footprints:TP_SMD_1mm, symbol antmicroTestPoints:TP_1mm_SMD
- removed U10, U11: TPD4E05U06QDQARQ1, antmicro-footprints:USON-10_2.5x1mm_P0.5mm, symbol antmicroTVSDiodes:TPD4E05U06QDQARQ1
Connections:
- no-connect marks 2 -> 1
Other:
- note removed: "HDMI"
- moved on the sheet: C129, J5, R80, R81, R82, R83, R84, R85, R86, R87, U12, U14
